File: ESP32 Base Design.kicad_sch (KiCad schematic)
At the start: 53 parts, among them J1 Conn_01x03_Pin, J2 Conn_01x03_Pin, J3 Conn_01x04_Pin, J4 Conn_01x04_Pin, T1 H1102NLT., U1 ESP32-S3, U2 W5500

Commit message: V2
Parts:
- removed J1, J2: Conn_01x03_Pin, symbol Connector:Conn_01x03_Pin
- removed J3: Conn_01x04_Pin, symbol Connector:Conn_01x04_Pin
- added C25, C9: 18pF, symbol Device:C
- added C26, C27: 12pF, symbol Device:C
- added C28: 22uF, symbol Device:C
- added C29, C42: 104, symbol Device:C
- added C30: 105, symbol Device:C
- added C31, C36: 22uF, symbol Device:C_Polarized
- added C32, C35: 104, symbol Device:C_Polarized
- added C33, C37, C38, C39, C40: 0.1uF, symbol Device:C
- added C34: 100P, symbol Device:C
- added C41: 1nF/2KV, symbol Device:C
- added D3: LED, symbol Device:LED
- added D4: 1N4148, Diode_THT:D_DO-35_SOD27_P7.62mm_Horizontal, symbol Diode:1N4148
- added J1: XLR5, symbol Connector_Audio:XLR5
- added J2: USB_C_Receptacle, symbol Connector:USB_C_Receptacle
- added J3: RJ45, symbol Connector:RJ45
- added J5: Conn_01x02_Pin, symbol Connector:Conn_01x02_Pin
- added J6: Conn_01x08, symbol Connector_Generic:Conn_01x08
- added L3: TBD, symbol Device:L
- added L4: 2.2uH/3A, symbol Device:L
- added Q1, Q2: NMOS, Package_TO_SOT_SMD:SOT-23, symbol Simulation_SPICE:NMOS
- added R10: 130R, Resistor_SMD:R_0603_1608Metric, symbol Device:R
- added R11, R9: 560R, Resistor_SMD:R_0603_1608Metric, symbol Device:R
- added R12, R13, R14: 3.3K, symbol Device:R
- added R31, R42: 1K, symbol Device:R
- added R32: 1M, symbol Device:R
- added R33: 0R, symbol Device:R
- added R34, R35: 30R, symbol Device:R
- added R36, R37: 5K1, symbol Device:R
- added R38, R39, R40: 10K, symbol Device:R
- added R4, R5, R6, R7: 10K, Resistor_SMD:R_0603_1608Metric, symbol Device:R
- added R41: 18K, symbol Device:R
- added R43, R44, R45, R46: 75R, symbol Device:R
- added R8: 4.7K, Resistor_SMD:R_0603_1608Metric, symbol Device:R
- added SW1, SW2, SW3, SW4, SW5, SW6: SW_Push, symbol Switch:SW_Push
- added U3: MAX3485, Package_SO:SOIC-8_3.9x4.9mm_P1.27mm, symbol Interface_UART:MAX3485
- added U4: W25Q128JVS, Package_SO:SOIC-8_5.3x5.3mm_P1.27mm, symbol Memory_Flash:W25Q128JVS
- added Y1: 40Mhz, symbol Device:Crystal_GND24
- added Y2: 25Mhz, symbol Device:Crystal_GND24
- C1, C12, C13, C14, C16, C18, C19, C2, C20, C21, C22, C23, C24, C3, C4, C5, C6, C7: footprint (none) -> Capacitor_SMD:C_0603_1608Metric
- C10, C11: footprint (none) -> Capacitor_SMD:C_1206_3216Metric
- C15, C17, C8: footprint (none) -> Capacitor_SMD:C_0805_2012Metric
- L1: footprint (none) -> Inductor_SMD:L_0603_1608Metric
- L2: value L -> 2.0nH
- R1, R15, R16, R17, R18, R19, R2, R20, R21, R22, R23, R24, R25, R26, R27, R28, R29, R3, R30: footprint (none) -> Resistor_SMD:R_0603_1608Metric
Connections:
- net +3V3: now also C29.1, C34.2, C35.1, C36.1, L4.2, Q1.2 (G), Q2.2 (G), R12.1, R13.1, R31.1, R38.1, R4.1, R40.2, R5.1, U4.8 (VCC)
- net ACTLED: now also U1.23 (GPIO17)
- net GND: now also C25.1, C26.1, C27.1, C28.2, C29.2, C30.2, C31.2, C32.2, C35.2, C36.2, C37.2, C38.2, C39.2, C40.2, C42.2, C9.1, D3.1 (K), J1.1 (P1), J2.A1 (GND), J2.A12 (GND), J2.B1 (GND), J2.B12 (GND), J2.S1 (SHIELD), J5.2 (Pin_2), R14.1, R36.1, R37.1, R41.1, SW1.2, SW2.2, SW3.2, SW4.2, SW5.2, SW6.2, U4.4 (GND), Y1.2, Y1.4, Y2.2, Y2.4
- net GP11: now also R25.1; no longer R28.1
- net GP12: now also R26.1; no longer R27.1
- net GP13: now also R27.1; no longer R26.1
- net GP14: now also R28.1; no longer R25.1
- net LINKLED: now also U1.24 (GPIO18); no longer J4.4 (Pin_4)
- net W_RD_OUT_N: now also C12.2, R21.2
- net W_RD_OUT_P: now also C13.2, R22.2
- net W_TD_OUT_N: now also R18.2, T1.3 (TD-)
- net W_TD_OUT_P: now also R20.2, T1.1 (TD+)
- net LED1_R: now reaches R15.1
- net LED1_R: now also U1.38 (GPIO33)
- net LED2_G: now reaches R2.2
- net LED2_G: now also U1.42 (GPIO37)
- net at C10.2, R21.1, R22.1: now also T1.7 (CT_2); no longer T1.15 (NC_6)
- net at U2.32 (~{SCS}): now also R28.2; no longer R25.2
- net at C12.1: now also T1.8 (RD-); no longer T1.16 (TX+)
- net W_RD_P: now reaches T1.11 (RX+)
- net W_RD_P: now also J3.3; no longer R18.2
- net W_RD_N: now reaches T1.9 (RX-)
- net W_RD_N: now also J3.6; no longer R20.2
- net RX: now reaches U1.10 (GPIO5)
- net RX: now also U3.1 (RO)
- net DIR_A: now reaches U1.11 (GPIO6)
- net DIR_A: now also Q2.3 (S), R5.2
- net TX_A: now reaches U1.12 (GPIO7)
- net TX_A: now also Q1.3 (S), R4.2
- net GPIO8: now reaches U1.13 (GPIO8)
- net GPIO8: now also J6.5 (Pin_5)
- net GP19: now reaches U1.25 (GPIO19/USB_D-)
- net GP19: now also R35.1
- net GP20: now reaches U1.26 (GPIO20/USB_D+)
- net GP20: now also R34.1
- net GPIO21: now reaches U1.27 (GPIO21)
- net GPIO21: now also J6.6 (Pin_6)
- net SPIHD: now reaches U1.30 (SPIHD)
- net SPIHD: now also U4.7 (~{HOLD}/~{RESET}/IO_{3})
- net SPIWP: now reaches U1.31 (SPIWP)
- net SPIWP: now also U4.3 (~{WP}/IO_{2})
- net SPICS0: now reaches U1.32 (SPICS0)
- net SPICS0: now also U4.1 (~{CS})
- net SPICLK: now reaches U1.33 (SPICLK)
- net SPICLK: now also U4.6 (CLK)
- net SPIQ: now reaches U1.34 (SPIQ)
- net SPIQ: now also U4.2 (DO/IO_{1})
- net SPID: now reaches U1.35 (SPID)
- net SPID: now also U4.5 (DI/IO_{0})
- net LED1_G: now reaches U1.39 (GPIO34)
- net LED1_G: now also R16.2
- net CHP_UP: now reaches U1.4 (CHIP_PU)
- net CHP_UP: now also C30.1, R38.2, SW5.1
- net LED1_B: now reaches U1.40 (GPIO35)
- net LED1_B: now also R17.1
- net LED2_R: now reaches U1.41 (GPIO36)
- net LED2_R: now also R3.1
- net LED2_B: now reaches U1.43 (GPIO38)
- net LED2_B: now also R1.1
- net GP0: now reaches U1.5 (GPIO0)
- net GP0: now also R13.2, SW6.1
- net GPIO45: now reaches U1.51 (GPIO45)
- net GPIO45: now also J6.8 (Pin_8)
- net GPIO46: now reaches U1.52 (GPIO46)
- net GPIO46: now also J6.7 (Pin_7)
- net GPIO1: now reaches U1.6 (GPIO1)
- net GPIO1: now also J6.1 (Pin_1)
- net GPIO2: now reaches U1.7 (GPIO2)
- net GPIO2: now also J6.2 (Pin_2)
- net GPIO3: now reaches U1.8 (GPIO3)
- net GPIO3: now also J6.3 (Pin_3)
- net GPIO4: now reaches U1.9 (GPIO4)
- net GPIO4: now also J6.4 (Pin_4)
- net at U2.30 (XI/CLKIN): now also R33.2
- net at U2.31 (XO): now also C9.2, R32.1, Y2.1
- net at U2.33 (SCLK): now also R27.2; no longer R26.2
- net at U2.34 (MISO): now also R26.2; no longer R27.2
- net at U2.35 (MOSI): now also R25.2; no longer R28.2
- net at C11.2, R19.2: now also T1.2 (CT_1); no longer T1.10 (NC_3)
- net at C13.1: now also T1.6 (RD+); no longer T1.14 (TX-)
- net MANUAL_B1 renamed W_VP
- net W_VP: now also J3.4, J3.5, R43.2
- net MANUAL_G1 renamed W_RXCM
- net W_RXCM: now also T1.10 (NC_3)
- net MANUAL_R1 renamed W_TXCM
- net W_TXCM: now also T1.15 (NC_6)
- net XTAL_N: no longer names the net of U1.53 (XTAL_N)
- net XTAL_N: now also C27.2, Y1.3
- net XTAL_P: no longer names the net of U1.54 (XTAL_P)
- net XTAL_P: now also L3.2
- new net: C42.1, R45.2, R46.2
- new net: J2.A5 (CC1), R36.2
- new net: J2.B5 (CC2), R37.2
- new net: C41.1, R43.1, R44.1, R45.1, R46.1
- new net: C34.1, R42.2
- new net: C25.2, R32.2, R33.1, Y2.3
- new net: Q1.1 (D), R7.2, R8.2, U3.4 (DI)
- new net: Q2.1 (D), R6.2, U3.2 (~{RE}), U3.3 (DE)
- new net: R9.1, U3.5 (GND)
- new net: R11.1, U3.8 (VCC)
- new net: C33.2, L4.1
- new net: C26.2, L3.1, Y1.1
- new net: D3.2 (A), R31.2
- new net: R40.1, R41.2, R42.1
- new net +3.3VA: R6.1, R7.1, R8.1
- new net +5V: C31.1, C32.1, D4.1 (K), R39.1
- new net 3V3_EN: R39.2
- new net A: J1.2 (P2), R10.2, R11.2, U3.7 (B)
- new net B: J1.3 (P3), R10.1, R9.2, U3.6 (A)
- new net DOWN_BTN: SW3.1
- new net GND2: C37.1, C38.1, C39.1, C40.1, C41.2
- new net GP15: R14.2
- new net LEFT_BTN: SW2.1
- new net RIGHT_BTN: SW1.1
- new net RST: R12.2
- new net UD_N: J2.A7 (D-), J2.B7 (D-), R35.2
- new net UD_P: J2.A6 (D+), J2.B6 (D+), R34.2
- new net UP_BTN: SW4.1
- new net VCOM: C28.1, D4.2 (A), J2.A4 (VBUS), J2.A9 (VBUS), J2.B4 (VBUS), J2.B9 (VBUS), J5.1 (Pin_1)
- new net W_TD_N: J3.2, T1.14 (TX-)
- new net W_TD_P: J3.1, T1.16 (TX+)
- new net W_VN: J3.7, J3.8, J4.4 (Pin_4), R44.2
Other:
- note added: "5PIN DMX"
- note added: "CONTROL"
- note added: "DEV GPIO"
- note added: "DISPLAY PROCCESSOR"
- note added: "DMX IC"
- note added: "FLASH"
- note added: "MAIN MCU"
- note added: "NETWORK INTERFACE"
- note added: "POE MODULE"
- note added: "POWER LED"
- note added: "PULLUPS"
- note added: "RESET CIRCUIT"
- note added: "USB C"
- note added: "USB POWER"
- moved on the sheet: C1, C10, C11, C12, C13, C14, C15, C16, C17, C18, C19, C2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
